Commit message: add kinect

File: abb_irb140_gazebo/urdf/irb140.xacro (robot description, xacro)
@@ -3,4 +3,9 @@
   <xacro:include filename="$(find abb_irb140_gazebo)/urdf/irb140_macro.xacro"/>
   <xacro:abb_irb140_g prefix=""/>
+  <xacro:include filename="$(find abb_irb140_support)/urdf/kinect_sensor.urdf.xacro"/>
+  <xacro:kinect_description prefix=""/>
+    <!--gazebo reference="kinect_joint">
+        <preserveFixedJoint>true</preserveFixedJoint>
+    </gazebo-->
   <!-- Fix robot to Gazebo world -->
   <link name="world"/>

File: abb_irb140_gazebo/urdf/irb140_macro.xacro (robot description, xacro)
@@ -9,5 +9,5 @@
     <type>transmission_interface/SimpleTransmission</type>
     <joint name="${prefix}joint_1">
-      <hardwareInterface>PositionJointInterface</hardwareInterface>
+      <hardwareInterface>hardware_interface/PositionJointInterface</hardwareInterface>
     </joint>
     <actuator name="${prefix}motor1">
@@ -18,5 +18,5 @@
     <type>transmission_interface/SimpleTransmission</type>
     <joint name="${prefix}joint_2">
-      <hardwareInterface>PositionJointInterface</hardwareInterface>
+      <hardwareInterface>hardware_interface/PositionJointInterface</hardwareInterface>
     </joint>
     <actuator name="${prefix}motor2">
@@ -27,5 +27,5 @@
     <type>transmission_interface/SimpleTransmission</type>
     <joint name="${prefix}joint_3">
-      <hardwareInterface>PositionJointInterface</hardwareInterface>
+      <hardwareInterface>hardware_interface/PositionJointInterface</hardwareInterface>
     </joint>
     <actuator name="${prefix}motor3">
@@ -36,5 +36,5 @@
     <type>transmission_interface/SimpleTransmission</type>
     <joint name="${prefix}joint_4">
-      <hardwareInterface>PositionJointInterface</hardwareInterface>
+      <hardwareInterface>hardware_interface/PositionJointInterface</hardwareInterface>
     </joint>
     <actuator name="${prefix}motor4">
@@ -45,5 +45,5 @@
     <type>transmission_interface/SimpleTransmission</type>
     <joint name="${prefix}joint_5">
-      <hardwareInterface>PositionJointInterface</hardwareInterface>
+      <hardwareInterface>hardware_interface/PositionJointInterface</hardwareInterface>
     </joint>
     <actuator name="${prefix}motor5">
@@ -54,5 +54,5 @@
     <type>transmission_interface/SimpleTransmission</type>
     <joint name="${prefix}joint_6">
-      <hardwareInterface>PositionJointInterface</hardwareInterface>
+      <hardwareInterface>hardware_interface/PositionJointInterface</hardwareInterface>
     </joint>
     <actuator name="${prefix}motor6">
@@ -90,4 +90,45 @@
     <turnGravityOff>true</turnGravityOff>
   </gazebo>
+  <!--gazebo reference="${camera_link_name}">
+    <sensor name="${camera_link_name}_camera" type="depth">
+        <update_rate>20</update_rate>
+        <camera>
+            <horizontal_fov>1.047198</horizontal_fov>
+            <image>
+                <width>640</width>
+                <height>480</height>
+                <format>R8G8B8</format>
+            </image>
+            <clip>
+                <near>0.05</near>
+                <far>3</far>
+            </clip>
+        </camera>
+        <plugin name="${camera_link_name}_controller" filename="libgazebo_ros_openni_kinect.so">
+            <baseline>0.2</baseline>
+            <alwaysOn>true</alwaysOn>
+            <updateRate>1.0</updateRate>
+            <cameraName>${camera_name}_ir</cameraName>
+            <imageTopicName>/${camera_name}/color/image_raw</imageTopicName>
+            <cameraInfoTopicName>/${camera_name}/color/camera_info</cameraInfoTopicName>
+            <depthImageTopicName>/${camera_name}/depth/image_raw</depthImageTopicName>
+            <depthImageInfoTopicName>/${camera_name}/depth/camera_info</depthImageInfoTopicName>
+            <pointCloudTopicName>/${camera_name}/depth/points</pointCloudTopicName>
+            <frameName>${frame_name}</frameName>
+            <pointCloudCutoff>0.5</pointCloudCutoff>
+            <pointCloudCutoffMax>3.0</pointCloudCutoffMax>
+            <distrotionK1>0.00000001</distrotionK1>
+            <distrotionK2>0.00000001</distrotionK2>
+            <distrotionK3>0.00000001</distrotionK3>
+            <distrotionT1>0.00000001</distrotionT1>
+            <distrotionT2>0.00000001</distrotionT2>
+            <CxPrime>0</CxPrime>
+            <Cx>0</Cx>
+            <Cy>0</Cy>
+            <focalLength>0</focalLength>
+            <hackBaseline>0</hackBaseline>
+        </plugin>
+    </sensor>
+  </gazebo-->
   <!-- ros_control plugin -->
   <gazebo>

File: abb_irb140_support/urdf/irb140.xacro (robot description, xacro)
@@ -3,3 +3,5 @@
 	<xacro:include filename="$(find abb_irb140_support)/urdf/irb140_macro.xacro"/>
 	<xacro:abb_irb140 prefix=""/>
+        <xacro:include filename="$(find abb_irb140_support)/urdf/kinect_sensor.urdf.xacro"/>
+        <xacro:kinect_description prefix=""/>
 </robot>

File: abb_irb140_support/urdf/irb140_macro.xacro (robot description, xacro)
@@ -6,15 +6,15 @@
     <inertial>
       <origin
-        xyz="0 0 0"
-        rpy="0 0 0" />
-      <mass
-        value="12" />
-      <inertia
-        ixx="1E-12"
-        ixy="1E-12"
-        ixz="1E-12"
-        iyy="1E-12"
-        iyz="1E-12"
-        izz="1E-12" />
+        xyz="-0.082039 0.00040203 0.059925"
+        rpy="0 0 0" />
+      <mass
+        value="96.79" />
+      <inertia
+        ixx="0.81512"
+        ixy="-7.8406E-05"
+        ixz="0.057274"
+        iyy="1.3048"
+        iyz="0.0065755"
+        izz="1.9226" />
     </inertial>
         <visual>
@@ -221,4 +221,23 @@
     </link>
     <link name="${prefix}tool0"/>
+    <!--link name="${prefix}kinect_link">
+        <visual>
+            <origin xyz="0 0 0" rpy="0 0 0"/>
+        </visual>
+    </link-->
+    <!--link name="${prefix}platform">
+        <visual>
+            <origin xyz="0 0 0" rpy="0 0 0"/>
+            <geometry>
+                <box size="0.5 0.5 1.0"/>
+            </geometry>
+            <material name="white"/>
+        </visual>
+        <collision>
+            <geometry>
+                <box size="0.5 0.5 1.0"/>
+            </geometry>
+        </collision>
+    </link-->
     <!-- end of link list -->
     <!-- joint list -->
@@ -270,4 +289,20 @@
         <origin xyz="0.05256 0 0" rpy="0 1.57079632679 0"/>
     </joint>
+    <!--joint name="${prefix}kinect_joint" type="fixed">
+        <origin xyz="0 -0.1 0" rpy="0 0 0"/>
+        <parent link="${prefix}link_5"/>
+        <child link="${prefix}kinect_link"/>
+    </joint-->
+    <!--joint name="${prefix}platform_joint" type="fixed">
+        <origin xyz="0.08 0 0.5" rpy="0 0 0"/>
+        <parent link="${prefix}platform"/>
+        <child link="${prefix}base_link"/>
+    </joint-->
+    <!--link name="${prefix}ground"/>
+    <joint name="${prefix}connnect_to_ground" type="fixed">
+        <orgign xyz="0 0 0.5" rpy="0 0 0"/>
+        <parent link="${prefix}ground"/>
+        <child link="${prefix}platform"/>
+    </joint-->
     <!-- end of joint list -->
     <!-- ROS base_link to ABB World Coordinates transform -->
